File: TeleRad.kicad_sch (KiCad schematic)
At the start: 9 parts, among them M1 Stepper_Motor_bipolar, M2 Stepper_Motor_bipolar

Commit message: Schematic update
Parts:
- added C3, C4: 100nF, symbol Device:C
- added U1: (no value), symbol Transformer:12V_to_3.3V_convertor
- C1, C2: value C -> 100uF
Connections:
- net +5V is gone; now on net Step2: ESP32-devkit-v1. (3.3V)
- net +12V: now also C3.2, C4.2, U1. (GND)
- net GND: now also C3.1, C4.1, U1. (GND)
- net Slp: no longer A2.13 (~{RST}), A2.14 (~{SLP})
- net ESP-3.3V renamed +3.3V
- net +3.3V: now also A2.13 (~{RST}), A2.14 (~{SLP}), U1. (GND)
- new net 12V: U1. (GND)
- no-connect marks 9 -> 10
Other:
- note added: "12V To 3.3V Buck"
- title: (none) -> TeleRad
- moved on the sheet: C2
